File: main board/Prototech-Farm/Schematic_V1.sch (EAGLE design)
At the start: 59 parts, among them Q1 SS8050-G, Q2 SS8050-G, Q3 SS8050-G, Q4 2n7000, Q5 2n7000, Q6 2n7000, Q7 2n7000, Q8 2n7000, SW1 MODE, SW2 RESET, U1 ESP32-WROOM-32U, U2 AMS1117-3.3, U3 ATTINY85-20PU, U4 ATTINY85-20PU, X1 pH_SNS, X10 SERVO1, X11 SERVO3, X12 SERVO5, X13 SERVO2, X14 SERVO4, X15 SERVO6, X16 I2C1, X17 I2C2, X18 I2C3, X19 I2C4, X2 EC_SNS, X3 TEMP_SNS, X4 Ultrasonic1, X5 Ultrasonic2, X6 Ultrasonic3, X7 Ultrasonic4, X8 Ultrasonic5, X9 RELAY_BLOCK

Commit message: DRC check board
Parts:
- added R20: 4k7, rcl:R-EU_M1206
Connections:
- net +5V: now also R20.2
- net TEMP_SNS0: now also R20.1
Changed lines of the file:
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@@
 <part name="R19" library="rcl" library_urn="urn:adsk.eagle:library:334" deviceset="R-EU_" device="M1206" package3d_urn="urn:adsk.eagle:package:23566/2" value="10k"/>
 <part name="Q8" library="BeagleBone_Blue_R3" library_urn="urn:adsk.eagle:library:5828899" deviceset="MOSFET-NCHANNEL" device="BSS138" package3d_urn="urn:adsk.eagle:package:5829571/1" value="2n7000"/>
+<part name="R20" library="rcl" library_urn="urn:adsk.eagle:library:334" deviceset="R-EU_" device="M1206" package3d_urn="urn:adsk.eagle:package:23566/2" value="4k7"/>
 </parts>
 <sheets>
@@
 <instance part="R19" gate="G$1" x="152.4" y="36.83" rot="R90"/>
 <instance part="Q8" gate="G$1" x="160.02" y="29.21" rot="MR270"/>
+<instance part="R20" gate="G$1" x="66.04" y="101.6" rot="R90"/>
 </instances>
 <busses>
@@
 <segment>
 <pinref part="X3" gate="-1" pin="S"/>
-<wire x1="44.45" y1="102.87" x2="49.53" y2="102.87" width="0.1524" layer="91"/>
 <pinref part="P+9" gate="1" pin="+5V"/>
 <wire x1="59.69" y1="127" x2="59.69" y2="123.19" width="0.1524" layer="91"/>
 <wire x1="59.69" y1="123.19" x2="59.69" y2="113.03" width="0.1524" layer="91"/>
-<wire x1="59.69" y1="113.03" x2="59.69" y2="102.87" width="0.1524" layer="91"/>
-<wire x1="59.69" y1="102.87" x2="49.53" y2="102.87" width="0.1524" layer="91"/>
+<wire x1="59.69" y1="113.03" x2="59.69" y2="106.68" width="0.1524" layer="91"/>
+<wire x1="59.69" y1="106.68" x2="59.69" y2="102.87" width="0.1524" layer="91"/>
+<wire x1="59.69" y1="102.87" x2="44.45" y2="102.87" width="0.1524" layer="91"/>
 <pinref part="X2" gate="-1" pin="S"/>
-<wire x1="44.45" y1="113.03" x2="49.53" y2="113.03" width="0.1524" layer="91"/>
-<wire x1="49.53" y1="113.03" x2="59.69" y2="113.03" width="0.1524" layer="91"/>
+<wire x1="44.45" y1="113.03" x2="59.69" y2="113.03" width="0.1524" layer="91"/>
 <junction x="59.69" y="113.03"/>
 <pinref part="X1" gate="-1" pin="S"/>
-<wire x1="44.45" y1="123.19" x2="49.53" y2="123.19" width="0.1524" layer="91"/>
-<wire x1="49.53" y1="123.19" x2="59.69" y2="123.19" width="0.1524" layer="91"/>
+<wire x1="44.45" y1="123.19" x2="59.69" y2="123.19" width="0.1524" layer="91"/>
 <junction x="59.69" y="123.19"/>
+<pinref part="R20" gate="G$1" pin="2"/>
+<wire x1="59.69" y1="106.68" x2="66.04" y2="106.68" width="0.1524" layer="91"/>
+<junction x="59.69" y="106.68"/>
 </segment>
 <segment>
@@
 <segment>
 <pinref part="X3" gate="-2" pin="S"/>
-<wire x1="44.45" y1="100.33" x2="49.53" y2="100.33" width="0.1524" layer="91"/>
 <label x="49.53" y="100.33" size="1.27" layer="95" xref="yes"/>
-</segment>
-<segment>
+<wire x1="44.45" y1="100.33" x2="59.69" y2="100.33" width="0.1524" layer="91"/>
+<wire x1="59.69" y1="100.33" x2="59.69" y2="96.52" width="0.1524" layer="91"/>
+<pinref part="R20" gate="G$1" pin="1"/>
+<wire x1="59.69" y1="96.52" x2="66.04" y2="96.52" width="0.1524" layer="91"/>
+</segment>
+<segment>
